File: Hardware/_autosave-GVH-POR-SpaceSuitScanner.kicad_pcb (KiCad board)
At the start: 2 copper layers, 68.1 x 221.9 mm, 53 parts, among them J1 Phoenix _725656, J10 Phoenix_5POS_1725685, J11 Phoenix _725656, J12 Phoenix _725656, J13 Phoenix _725656, J14 Phoenix _725656, J15 Phoenix _725656, J16 Phoenix _725656, J17 Phoenix _725656, J18 Phoenix _725656, J19 Phoenix_3POS_1725669, J2 Phoenix _725656, J29 n00d i2c, J3 Phoenix _725656, J30 Matrix i2c, J31 Speaker In, J32 Speaker, J4 Phoenix _725656, J5 Phoenix _725656, J6 Phoenix _725656, J7 Phoenix _725656, J8 Phoenix _725656, J9 Phoenix _725656, K1 EC2-3NU, Q1 Q_NPN_BEC, U1 AW9523, U2 AW9523, U3 AW9523 Expander, U4 AW9523 Expander, U5 AT42QT1010, U6 IS31FL3731 LED Driver

Commit message: Schematic progress
Routing:
- net VCC: track 4.47 -> 0.00 mm
- net GND: track 0.00 -> 2.67 mm
Changed lines of the file:
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@@
   (gr_curve (pts (xy 59.864744 41.024202) (xy 59.864744 41.024262) (xy 59.864744 41.024321) (xy 59.864744 41.024381))
     (stroke (width 0.25) (type solid)) (layer "F.Fab"))
-  (segment (start 98.295208 169.418) (end 99.709421 169.418) (width 0.2) (layer "F.Cu") (net 1))
-  (segment (start 99.709421 169.418) (end 99.822 169.418) (width 0.2) (layer "F.Cu") (net 1))
-  (segment (start 98.314283 168.022862) (end 99.709421 169.418) (width 0.2) (layer "F.Cu") (net 1))
-  (segment (start 97.607177 168.729969) (end 98.295208 169.418) (width 0.2) (layer "F.Cu") (net 1))
+  (segment (start 97.7775 180.8355) (end 97.79 180.848) (width 0.254) (layer "F.Cu") (net 2))
+  (segment (start 97.7775 180.779239) (end 97.7775 180.8355) (width 0.254) (layer "F.Cu") (net 2))
+  (segment (start 97.7775 180.8355) (end 97.7775 178.239239) (width 0.254) (layer "F.Cu") (net 2))
   (segment (start 103.09 171.889239) (end 100.056511 171.889239) (width 0.254) (layer "F.Cu") (net 9))
   (segment (start 100.056511 171.889239) (end 97.252208 169.084936) (width 0.254) (layer "F.Cu") (net 9))
