File: Hardware/GVH-POR-SpaceSuitScanner.kicad_pcb (KiCad board)
At the start: 2 copper layers, 68.1 x 221.9 mm, 53 parts, among them J1 Phoenix _725656, J10 Phoenix_5POS_1725685, J11 Phoenix _725656, J12 Phoenix _725656, J13 Phoenix _725656, J14 Phoenix _725656, J15 Phoenix _725656, J16 Phoenix _725656, J17 Phoenix _725656, J18 Phoenix _725656, J19 Phoenix_3POS_1725669, J2 Phoenix _725656, J29 n00d i2c, J3 Phoenix _725656, J30 Matrix i2c, J31 Speaker In, J32 Speaker, J4 Phoenix _725656, J5 Phoenix _725656, J6 Phoenix _725656, J7 Phoenix _725656, J8 Phoenix _725656, J9 Phoenix _725656, K1 EC2-3NU, Q1 Q_NPN_BEC, U1 AW9523, U2 AW9523, U3 AW9523 Expander, U4 AW9523 Expander, U5 AT42QT1010, U6 IS31FL3731 LED Driver

Commit message: Continuing PCB Layout Process
Parts:
- removed D2: 1N4148, Diode_SMD:D_SOD-123
- removed D3: LED, LED_SMD:LED_0805_2012Metric_Pad1.15x1.40mm_HandSolder
- removed K1: EC2-3NU, my_footprints:RELAY8_EE2-3NUH_KEM-M
- removed Q1: Q_NPN_BEC, Package_TO_SOT_SMD:SOT-23
- removed R5, R7: 1K, Resistor_SMD:R_0805_2012Metric
- removed R6: 10K, Resistor_SMD:R_0805_2012Metric
- D4, D5: footprint LED_SMD:LED_0805_2012Metric_Pad1.15x1.40mm_HandSolder -> LED_THT:LED_Rectangular_W5.0mm_H2.0mm
- moved J18 188.0 mm to (56.1, 220.2), turned to -90 degrees
- moved J19 179.4 mm to (53.0, 228.8), turned to -90 degrees
- moved J17 175.6 mm to (56.1, 210.0), turned to -90 degrees
- moved J14 169.5 mm to (56.1, 179.5), turned to -90 degrees
- moved J16 163.5 mm to (56.1, 199.8), turned to -90 degrees
- moved J13 158.1 mm to (56.1, 169.4), turned to -90 degrees
- moved J15 151.5 mm to (56.1, 189.7), turned to -90 degrees
- moved J9 151.0 mm to (56.1, 118.6), turned to -90 degrees
- moved J5 148.2 mm to (56.1, 77.9), turned to -90 degrees
- moved J12 146.9 mm to (56.1, 159.2), turned to -90 degrees
- moved J8 141.9 mm to (56.1, 108.4), turned to -90 degrees
- moved J4 141.3 mm to (56.1, 67.8), turned to -90 degrees
- moved J11 135.9 mm to (56.1, 149.0), turned to -90 degrees
- moved J3 135.3 mm to (56.1, 57.6), turned to -90 degrees
- moved J7 133.6 mm to (56.1, 100.8), turned to -90 degrees
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Connections:
- U4 pad 1: P02_0 -> P02_1
Routing:
- net P02_1: track 0.00 -> 13.8 mm
- net P02_0: track 0.00 -> 13.7 mm
- net P12_7: track 0.00 -> 12.8 mm
- net P12_3: track 0.00 -> 11.4 mm
- net P02_2: track 0.00 -> 11.0 mm
- net P12_6: track 0.00 -> 10.4 mm
- net P12_2: track 0.00 -> 9.05 mm
- net P02_3: track 0.00 -> 8.63 mm
- net P12_5: track 0.00 -> 8.09 mm
- net NOOD_SCL: track 8.26 -> 16.3 mm
- net NOOD_SDA: track 7.00 -> 13.8 mm
- net P02_4: track 0.00 -> 6.76 mm
- net P12_1: track 0.00 -> 6.71 mm
- net P12_4: track 0.00 -> 6.16 mm
- net P02_5: track 0.00 -> 5.50 mm
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
Commit message: Finished laying out PCB
Parts:
- added C7: 22nF, Connector_PinHeader_2.54mm:PinHeader_1x02_P2.54mm_Vertical, F.Cu at (64.5, 139.7)
- added G***: LOGO, MeowWolf_Logos:MW_Logo_Horizontal_3.0inch, F.Cu at (374.0, 243.8)
- moved R2 65.8 mm to (74.9, 171.7), turned to 90 degrees
- moved R1 62.3 mm to (79.7, 179.1)
- moved JP1 22.6 mm to (108.5, 217.2)
- moved R8 22.6 mm to (108.5, 213.5)
- moved JP2 18.4 mm to (112.4, 217.2)
- moved R9 18.4 mm to (112.6, 213.5)
- moved C3 5.22 mm to (83.6, 159.2), turned to 90 degrees
- moved C4 5.22 mm to (86.1, 159.2), turned to 90 degrees
- moved C1 5.21 mm to (83.6, 179.5), turned to 90 degrees
- moved C2 5.21 mm to (86.1, 179.5), turned to 90 degrees
- moved R4 4.94 mm to (73.7, 146.1), turned to 90 degrees
- moved D1 4.19 mm to (73.7, 141.0), turned to 90 degrees
- moved C6 3.77 mm to (68.6, 145.0)
- moved U5 3.77 mm to (68.6, 141.1)
- moved J29 0.30 mm to (69.8, 203.2)
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Connections:
- D1 pad 2: TOUCH_OUT -> P11_0
- J1 pad 1: unconnected-(J1-Pad1) -> P01_1
- J1 pad 2: unconnected-(J1-Pad2) -> P01_2
- J10 pad 1: unconnected-(J10-Pad1) -> P11_1
- J10 pad 3: unconnected-(J10-Pad3) -> CAP_WIRE
- J10 pad 5: unconnected-(J10-Pad5) -> P02_7
- J11 pad 2: unconnected-(J11-Pad2) -> P12_4
- J12 pad 2: unconnected-(J12-Pad2) -> P12_5
- J13 pad 1: unconnected-(J13-Pad1) -> P12_6
- J13 pad 2: unconnected-(J13-Pad2) -> P12_7
- J14 pad 2: unconnected-(J14-Pad2) -> P02_6
- J15 pad 2: unconnected-(J15-Pad2) -> P02_5
- J16 pad 2: unconnected-(J16-Pad2) -> P02_4
- J17 pad 2: unconnected-(J17-Pad2) -> P02_3
- J18 pad 2: unconnected-(J18-Pad2) -> P02_2
- J19 pad 1: unconnected-(J19-Pad1) -> VCC
- J19 pad 2: unconnected-(J19-Pad2) -> P02_1
- J19 pad 3: unconnected-(J19-Pad3) -> P12_0
- J2 pad 2: unconnected-(J2-Pad2) -> P01_3
- J3 pad 2: unconnected-(J3-Pad2) -> P01_4
- J4 pad 2: unconnected-(J4-Pad2) -> P01_5
- J5 pad 2: unconnected-(J5-Pad2) -> P01_6
- J6 pad 2: unconnected-(J6-Pad2) -> P01_7
- J7 pad 1: unconnected-(J7-Pad1) -> P11_4
- J7 pad 2: unconnected-(J7-Pad2) -> P11_5
- J8 pad 2: unconnected-(J8-Pad2) -> P11_6
- J9 pad 2: unconnected-(J9-Pad2) -> P11_7
- JP1 pad 1: Net-(JP1-A) -> P12_3
- JP2 pad 1: Net-(JP2-A) -> P02_0
- R3 pad 1: unconnected-(R3-Pad1) -> Net-(U5-SNSK)
- R3 pad 2: Net-(U5-SNSK) -> CAP_WIRE
- R8 pad 1: Net-(JP1-A) -> P12_3
- R9 pad 1: Net-(JP2-A) -> P02_0
- U5 pad 1: TOUCH_OUT -> P11_0
Routing:
- net VCC: track 0.00 -> 456.0 mm, vias 0 -> 2
- net MATRIX_SDA: track 0.00 -> 203.1 mm, vias 0 -> 1
- net MATRIX_SCL: track 0.00 -> 199.8 mm, vias 0 -> 1
- net P01_1: track 14.4 -> 189.0 mm
- net P01_2: track 10.9 -> 182.9 mm
- net P01_3: track 8.54 -> 176.2 mm
- net P01_4: track 6.54 -> 162.7 mm
- net P01_5: track 5.28 -> 145.4 mm
- net P01_7: track 4.68 -> 140.0 mm
- net P01_6: track 4.02 -> 138.4 mm
- net P11_4: track 5.94 -> 126.5 mm
- net P11_5: track 8.00 -> 126.3 mm
- net GND: track 0.00 -> 102.9 mm, vias 0 -> 10
- net P11_6: track 10.3 -> 103.1 mm
- net P02_1: track 13.8 -> 105.6 mm
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- added copper zone on B.Cu, net GND
- added copper zone on F.Cu, net GND
Other:
- board text added: "+"
- board text added: "Green"
- board text added: "Matrix i2c"
- board text added: "Noodle i2c"
- board text added: "SCL"
- board text added: "SDA"
- board text added: "Speaker"
