File: Hardware/GVH-POR-SpaceSuitScanner.kicad_pcb (KiCad board)
At the start: 2 copper layers, 68.1 x 221.9 mm, 48 parts, among them J1 Phoenix _725656, J10 Phoenix_5POS_1725685, J11 Phoenix _725656, J12 Phoenix _725656, J13 Phoenix _725656, J14 Phoenix _725656, J15 Phoenix _725656, J16 Phoenix _725656, J17 Phoenix _725656, J18 Phoenix _725656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

Commit message: Added pull down resistor to touch output
Parts:
- added R5: 10K, Resistor_SMD:R_0805_2012Metric, F.Cu at (79.1, 144.4)
Routing:
- net P11_0: track 49.3 -> 52.2 mm
Changed lines of the file:
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@@
       (net 42 "P12_7") (pinfunction "2") (pintype "passive") (solder_mask_margin 0.102))
+  )
+  (footprint "Resistor_SMD:R_0805_2012Metric" (layer "F.Cu")
+    (at 79.0975 144.4225 -90)
+    (descr "Resistor SMD 0805 (2012 Metric), square (rectangular) end terminal, IPC_7351 nominal, (Body size source: IPC-SM-782 page 72, https://www.pcb-3d.com/wordpress/wp-content/uploads/ipc-sm-782a_amendment_1_and_2.pdf), generated with kicad-footprint-generator")
+    (tags "resistor")
+    (property "Sheetfile" "GVH-POR-SpaceSuitScanner.kicad_sch")
+    (property "Sheetname" "")
+    (property "ki_description" "Resistor, small symbol")
+    (property "ki_keywords" "R resistor")
+    (attr smd)
+    (fp_text reference "R5" (at 0 -1.65 90) (layer "F.SilkS")
+        (effects (font (size 1 1) (thickness 0.15)))
+    )
+    (fp_text value "10K" (at 0 1.65 90) (layer "F.Fab")
+        (effects (font (size 1 1) (thickness 0.15)))
+    )
+    (fp_text user "${REFERENCE}" (at 0 0 90) (layer "F.Fab")
+        (effects (font (size 0.5 0.5) (thickness 0.08)))
+    )
+    (fp_line (start -0.227064 -0.735) (end 0.227064 -0.735)
+      (stroke (width 0.12) (type solid)) (layer "F.SilkS"))
+    (fp_line (start -0.227064 0.735) (end 0.227064 0.735)
+      (stroke (width 0.12) (type solid)) (layer "F.SilkS"))
+    (fp_line (start -1.68 -0.95) (end 1.68 -0.95)
+      (stroke (width 0.05) (type solid)) (layer "F.CrtYd"))
+    (fp_line (start -1.68 0.95) (end -1.68 -0.95)
+      (stroke (width 0.05) (type solid)) (layer "F.CrtYd"))
+    (fp_line (start 1.68 -0.95) (end 1.68 0.95)
+      (stroke (width 0.05) (type solid)) (layer "F.CrtYd"))
+    (fp_line (start 1.68 0.95) (end -1.68 0.95)
+      (stroke (width 0.05) (type solid)) (layer "F.CrtYd"))
+    (fp_line (start -1 -0.625) (end 1 -0.625)
+      (stroke (width 0.1) (type solid)) (layer "F.Fab"))
+    (fp_line (start -1 0.625) (end -1 -0.625)
+      (stroke (width 0.1) (type solid)) (layer "F.Fab"))
+    (fp_line (start 1 -0.625) (end 1 0.625)
+      (stroke (width 0.1) (type solid)) (layer "F.Fab"))
+    (fp_line (start 1 0.625) (end -1 0.625)
+      (stroke (width 0.1) (type solid)) (layer "F.Fab"))
+    (pad "1" smd roundrect (at -0.9125 0 270) (size 1.025 1.4) (layers "F.Cu" "F.Paste" "F.Mask") (roundrect_rratio 0.243902)
+      (net 12 "P11_0") (pintype "passive"))
+    (pad "2" smd roundrect (at 0.9125 0 270) (size 1.025 1.4) (layers "F.Cu" "F.Paste" "F.Mask") (roundrect_rratio 0.243902)
+      (net 2 "GND") (pintype "passive"))
+    (model "${KICAD6_3DMODEL_DIR}/Resistor_SMD.3dshapes/R_0805_2012Metric.wrl"
+      (offset (xyz 0 0 0))
+      (scale (xyz 1 1 1))
+      (rotate (xyz 0 0 0))
+    )
   )
   (footprint "my_footprints:PHOENIX_1725656-2POS" (layer "F.Cu")
@@
   (segment (start 95.429 163.614897) (end 95.429 165.39713) (width 0.254) (layer "F.Cu") (net 12))
   (segment (start 92.78907 160.974967) (end 95.429 163.614897) (width 0.254) (layer "F.Cu") (net 12))
+  (segment (start 76.2 143.51) (end 79.0975 143.51) (width 0.254) (layer "F.Cu") (net 12))
   (segment (start 69.53 139.9) (end 73.615 139.9) (width 0.254) (layer "F.Cu") (net 12))
   (segment (start 76.2 143.51) (end 76.2 142.485) (width 0.254) (layer "F.Cu") (net 12))

Commit message: Backing up again
Routing:
- net P01_3: track 176.2 -> 174.9 mm
Changed lines of the file:
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@@
   (segment (start 88.138 181.229) (end 89.535 182.626) (width 0.254) (layer "B.Cu") (net 1))
   (segment (start 97.79 175.26) (end 99.06 173.99) (width 0.254) (layer "F.Cu") (net 2))
-  (segment (start 99.106068 153.623932) (end 99.106068 152.576953) (width 0.254) (layer "F.Cu") (net 2))
   (segment (start 92.409 179.5272) (end 92.762553 179.5272) (width 0.254) (layer "F.Cu") (net 2))
   (segment (start 92.02893 160.974967) (end 91.44 161.563897) (width 0.254) (layer "F.Cu") (net 2))
   (segment (start 97.029753 175.26) (end 97.79 175.26) (width 0.254) (layer "F.Cu") (net 2))
-  (segment (start 99.106068 152.576953) (end 101.823021 149.86) (width 0.254) (layer "F.Cu") (net 2))
   (segment (start 110.49 153.67) (end 110.49 157.48) (width 0.254) (layer "F.Cu") (net 2))
   (segment (start 78.74 156.21) (end 74.93 160.02) (width 0.254) (layer "F.Cu") (net 2))
@@
   (segment (start 81.28 156.21) (end 78.74 156.21) (width 0.254) (layer "F.Cu") (net 2))
   (segment (start 93.84973 178.440023) (end 97.029753 175.26) (width 0.254) (layer "F.Cu") (net 2))
-  (segment (start 94.053469 157.536214) (end 95.193786 157.536214) (width 0.254) (layer "F.Cu") (net 2))
   (segment (start 90.261163 158.44706) (end 88.024103 156.21) (width 0.254) (layer "F.Cu") (net 2))
-  (segment (start 93.84973 157.739953) (end 94.053469 157.536214) (width 0.254) (layer "F.Cu") (net 2))
+  (segment (start 101.823021 149.86) (end 106.68 149.86) (width 0.254) (layer "F.Cu") (net 2))
   (segment (start 82.729 185.8772) (end 82.729 187.781) (width 1.27) (layer "F.Cu") (net 2))
   (segment (start 92.02893 181.675037) (end 91.44 182.263967) (width 0.254) (layer "F.Cu") (net 2))
@@
   (segment (start 82.729 187.781) (end 81.28 189.23) (width 1.27) (layer "F.Cu") (net 2))
   (segment (start 92.762553 158.82713) (end 93.84973 157.739953) (width 0.254) (layer "F.Cu") (net 2))
-  (segment (start 101.823021 149.86) (end 106.68 149.86) (width 0.254) (layer "F.Cu") (net 2))
   (segment (start 99.06 173.99) (end 99.06 168.91) (width 0.254) (layer "F.Cu") (net 2))
-  (segment (start 106.68 149.86) (end 110.49 153.67) (width 0.254) (layer "F.Cu") (net 2))
+  (segment (start 96.2406 156.9974) (end 99.106068 154.131932) (width 0.254) (layer "F.Cu") (net 2))
   (segment (start 92.762553 179.5272) (end 93.84973 178.440023) (width 0.254) (layer "F.Cu") (net 2))
   (segment (start 91.44 161.563897) (end 91.44 170.18) (width 0.254) (layer "F.Cu") (net 2))
-  (segment (start 95.193786 157.536214) (end 99.106068 153.623932) (width 0.254) (layer "F.Cu") (net 2))
+  (segment (start 106.68 149.86) (end 110.49 153.67) (width 0.254) (layer "F.Cu") (net 2))
+  (segment (start 94.592283 156.9974) (end 96.2406 156.9974) (width 0.254) (layer "F.Cu") (net 2))
+  (segment (start 99.106068 152.576953) (end 101.823021 149.86) (width 0.254) (layer "F.Cu") (net 2))
+  (segment (start 99.106068 154.131932) (end 99.106068 152.576953) (width 0.254) (layer "F.Cu") (net 2))
+  (segment (start 93.84973 157.739953) (end 94.592283 156.9974) (width 0.254) (layer "F.Cu") (net 2))
   (via (at 67.31 152.4) (size 0.8) (drill 0.4) (layers "F.Cu" "B.Cu") (net 2))
   (via (at 85.09 162.56) (size 0.8) (drill 0.4) (layers "F.Cu" "B.Cu") (free) (net 2))
@@
   (segment (start 104.61613 151.13) (end 113.03 151.13) (width 0.254) (layer "B.Cu") (net 17))
   (segment (start 103.049 152.69713) (end 104.61613 151.13) (width 0.254) (layer "B.Cu") (net 17))
-  (segment (start 94.406576 157.890214) (end 97.355284 157.890214) (width 0.254) (layer "F.Cu") (net 18))
+  (segment (start 96.566986 157.890214) (end 100.509 153.9482) (width 0.254) (layer "F.Cu") (net 18))
+  (segment (start 100.509 153.9482) (end 100.509 152.69713) (width 0.254) (layer "F.Cu") (net 18))
   (segment (start 94.203283 158.093507) (end 94.406576 157.890214) (width 0.254) (layer "F.Cu") (net 18))
-  (segment (start 100.509 154.736498) (end 100.509 152.69713) (width 0.254) (layer "F.Cu") (net 18))
-  (segment (start 100.509 152.69713) (end 99.59966 152.69713) (width 0.254) (layer "F.Cu") (net 18))
-  (segment (start 97.355284 157.890214) (end 100.509 154.736498) (width 0.254) (layer "F.Cu") (net 18))
+  (segment (start 94.406576 157.890214) (end 96.566986 157.890214) (width 0.254) (layer "F.Cu") (net 18))
   (segment (start 105.8672 49.9872) (end 56.059 49.9872) (width 0.254) (layer "B.Cu") (net 18))
   (segment (start 100.509 152.69713) (end 103.34613 149.86) (width 0.254) (layer "B.Cu") (net 18))

Commit message: PCB Ordered. First version of design archived
Parts:
- removed C1, C3: 10uF, Capacitor_SMD:C_0805_2012Metric_Pad1.18x1.45mm_HandSolder
- removed C2, C4: 0.1uF, Capacitor_SMD:C_0805_2012Metric_Pad1.18x1.45mm_HandSolder
- removed the G*** at (374.0, 243.8)
- removed R1, R2: 10k, Resistor_SMD:R_0805_2012Metric_Pad1.20x1.40mm_HandSolder
- removed U1, U2: AW9523, Package_DFN_QFN:TQFN-24-1EP_4x4mm_P0.5mm_EP2.6x2.6mm
- added G***: LOGO, MeowWolf_Logos:MW_Logo_Horizontal_1.0inch, F.Cu at (83.8, 212.3)
- added G***: LOGO, MeowWolf_Logos:MW_Mark_0.50inch, F.Cu at (83.8, 52.3)
- moved D1 19.9 mm to (65.7, 159.2)
- moved R4 19.9 mm to (65.7, 164.3)
- moved R5 19.9 mm to (71.1, 162.7)
- moved C6 1.30 mm to (67.6, 145.8)
Routing:
- net GND: track 103.2 -> 0.00 mm, vias 10 -> 2
- net VCC: track 456.0 -> 398.4 mm, vias 2 -> 4
- net P01_1: track 189.0 -> 161.1 mm
- net P01_2: track 182.9 -> 159.1 mm
- net P01_3: track 174.9 -> 154.1 mm
- net P11_7: track 99.7 -> 82.1 mm
- net P11_5: track 126.3 -> 111.5 mm
- net P11_6: track 103.1 -> 88.4 mm
- net P11_4: track 126.5 -> 112.0 mm
- net P01_0: track 13.8 -> 0.00 mm
- net P02_0: track 47.5 -> 34.0 mm
- net P01_4: track 162.7 -> 149.2 mm
- net P12_7: track 37.4 -> 24.7 mm
- net P01_7: track 140.0 -> 128.1 mm
- net P11_3: track 11.5 -> 0.00 mm
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Other:
- board text added: "GVH • Darlu's Spacesuit Activator • V0.2 Daniel Bornhorst • 08/2024"
