File: Hardware/GVH-POR-SpaceSuitScanner.kicad_sch (KiCad schematic)
At the start: 48 parts, among them J1 Phoenix _725656, J10 Phoenix_5POS_1725685, J11 Phoenix _725656, J12 Phoenix _725656, J13 Phoenix _725656, J14 Phoenix _725656, J15 Phoenix _725656, J16 Phoenix _725656, J17 Phoenix _725656, J18 Phoenix _725656, J19 Phoenix_3POS_1725669, J2 Phoenix _725656, J29 n00d i2c, J3 Phoenix _725656, J30 Matrix i2c, J31 Speaker In, J32 Speaker, J4 Phoenix _725656, J5 Phoenix _725656, J6 Phoenix _725656, J7 Phoenix _725656, J8 Phoenix _725656, J9 Phoenix _725656, U1 AW9523, U2 AW9523, U3 AW9523 Expander, U4 AW9523 Expander, U5 AT42QT1010, U6 IS31FL3731 LED Driver

Commit message: Added pull down resistor to touch output
Parts:
- added R5: 10K, Resistor_SMD:R_0805_2012Metric, symbol Device:R_Small
Connections:
- net GND: now also R5.2
- net P11_0: now also R5.1
Other:
- note added: "Pull down resistor"
- moved on the sheet: D1, R4
Changed lines of the file:
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@@
     (stroke (width 0) (type default))
   )
+  (wire (pts (xy 198.12 187.96) (xy 201.93 187.96))
+    (stroke (width 0) (type default))
+  )
   (wire (pts (xy 191.77 95.25) (xy 194.31 95.25))
     (stroke (width 0) (type default))
@@
     (stroke (width 0) (type default))
   )
-  (wire (pts (xy 139.7 195.58) (xy 146.05 195.58))
+  (wire (pts (xy 139.7 198.12) (xy 146.05 198.12))
     (stroke (width 0) (type default))
   )
@@
     (stroke (width 0) (type default))
   )
-  (wire (pts (xy 171.45 198.12) (xy 171.45 195.58))
+  (wire (pts (xy 171.45 200.66) (xy 171.45 198.12))
     (stroke (width 0) (type default))
   )
@@
     (stroke (width 0) (type default))
   )
-  (wire (pts (xy 171.45 195.58) (xy 163.83 195.58))
+  (wire (pts (xy 171.45 198.12) (xy 163.83 198.12))
     (stroke (width 0) (type default))
   )
@@
     (stroke (width 0) (type default))
   )
-  (wire (pts (xy 151.13 195.58) (xy 158.75 195.58))
+  (wire (pts (xy 151.13 198.12) (xy 158.75 198.12))
     (stroke (width 0) (type default))
   )
@@
     (stroke (width 0) (type default))
   )
+  (wire (pts (xy 207.01 187.96) (xy 212.09 187.96))
+    (stroke (width 0) (type default))
+  )
   (wire (pts (xy 106.68 36.83) (xy 109.22 36.83))
     (stroke (width 0) (type default))
@@
     (stroke (width 0) (type default))
   )
+  (wire (pts (xy 212.09 187.96) (xy 212.09 190.5))
+    (stroke (width 0) (type default))
+  )
   (wire (pts (xy 106.68 24.13) (xy 106.68 25.4))
     (stroke (width 0) (type default))
@@
     (effects (font (size 1.27 1.27)) (justify left bottom))
   )
+  (text "Pull down resistor" (at 186.69 191.77 0)
+    (effects (font (size 1.27 1.27)) (justify left bottom))
+  )
   (text "I2C Pullup resistors\n" (at 44.45 20.32 0)
     (effects (font (size 1.27 1.27)) (justify left bottom))
@@
     )
   )
+  (global_label "TOUCH_OUT" (shape input) (at 198.12 187.96 180) (fields_autoplaced)
+    (effects (font (size 1.27 1.27)) (justify right))
+    (property "Intersheetrefs" "${INTERSHEET_REFS}" (at 184.3095 187.96 0)
+      (effects (font (size 1.27 1.27)) (justify right) hide)
+    )
+  )
   (global_label "P01_6" (shape input) (at 142.24 116.84 0) (fields_autoplaced)
     (effects (font (size 1.27 1.27)) (justify left))
@@
     )
   )
-  (global_label "TOUCH_OUT" (shape input) (at 139.7 195.58 180) (fields_autoplaced)
+  (global_label "TOUCH_OUT" (shape input) (at 139.7 198.12 180) (fields_autoplaced)
     (effects (font (size 1.27 1.27)) (justify right))
-    (property "Intersheetrefs" "${INTERSHEET_REFS}" (at 125.8895 195.58 0)
+    (property "Intersheetrefs" "${INTERSHEET_REFS}" (at 125.8895 198.12 0)
       (effects (font (size 1.27 1.27)) (justify right) hide)
     )
@@
     )
   )
-  (symbol (lib_id "Device:LED_Small") (at 148.59 195.58 180) (unit 1)
+  (symbol (lib_id "Device:LED_Small") (at 148.59 198.12 180) (unit 1)
     (in_bom yes) (on_board yes) (dnp no) (fields_autoplaced)
-    (property "Reference" "D1" (at 148.5265 189.23 0)
+    (property "Reference" "D1" (at 148.5265 191.77 0)
       (effects (font (size 1.27 1.27)))
     )
-    (property "Value" "LED_Small" (at 148.5265 191.77 0)
+    (property "Value" "LED_Small" (at 148.5265 194.31 0)
       (effects (font (size 1.27 1.27)))
     )
-    (property "Footprint" "LED_SMD:LED_0805_2012Metric_Pad1.15x1.40mm_HandSolder" (at 148.59 195.58 90)
+    (property "Footprint" "LED_SMD:LED_0805_2012Metric_Pad1.15x1.40mm_HandSolder" (at 148.59 198.12 90)
       (effects (font (size 1.27 1.27)) hide)
     )
-    (property "Datasheet" "~" (at 148.59 195.58 90)
+    (property "Datasheet" "~" (at 148.59 198.12 90)
       (effects (font (size 1.27 1.27)) hide)
     )
@@
     )
   )
-  (symbol (lib_id "power:GND") (at 171.45 198.12 0) (unit 1)
+  (symbol (lib_id "power:GND") (at 171.45 200.66 0) (unit 1)
     (in_bom yes) (on_board yes) (dnp no) (fields_autoplaced)
-    (property "Reference" "#PWR021" (at 171.45 204.47 0)
+    (property "Reference" "#PWR021" (at 171.45 207.01 0)
       (effects (font (size 1.27 1.27)) hide)
     )
-    (property "Value" "GND" (at 171.45 203.2 0)
+    (property "Value" "GND" (at 171.45 205.74 0)
       (effects (font (size 1.27 1.27)))
     )
-    (property "Footprint" "" (at 171.45 198.12 0)
+    (property "Footprint" "" (at 171.45 200.66 0)
       (effects (font (size 1.27 1.27)) hide)
     )
-    (property "Datasheet" "" (at 171.45 198.12 0)
+    (property "Datasheet" "" (at 171.45 200.66 0)
       (effects (font (size 1.27 1.27)) hide)
     )
@@
     )
   )
+  (symbol (lib_id "power:GND") (at 212.09 190.5 0) (unit 1)
+    (in_bom yes) (on_board yes) (dnp no) (fields_autoplaced)
+    (property "Reference" "#PWR023" (at 212.09 196.85 0)
+      (effects (font (size 1.27 1.27)) hide)
+    )
+    (property "Value" "GND" (at 212.09 195.58 0)
+      (effects (font (size 1.27 1.27)))
+    )
+    (property "Footprint" "" (at 212.09 190.5 0)
+      (effects (font (size 1.27 1.27)) hide)
+    )
+    (property "Datasheet" "" (at 212.09 190.5 0)
+      (effects (font (size 1.27 1.27)) hide)
+    )
+    (pin "1")
+    (instances
+      (project "GVH-POR-SpaceSuitScanner"
+        (path "/d220c84c-6011-402a-bba2-62b84e1ad1c6"
+          (reference "#PWR023") (unit 1)
+        )
+      )
+    )
+  )
   (symbol (lib_id "my_library:Phoenix_2POS_725656") (at 312.42 33.02 0) (unit 1)
     (in_bom yes) (on_board yes) (dnp no) (fields_autoplaced)
@@
     )
   )
+  (symbol (lib_id "Device:R_Small") (at 204.47 187.96 90) (mirror x) (unit 1)
+    (in_bom yes) (on_board yes) (dnp no)
+    (property "Reference" "R5" (at 204.47 182.88 90)
+      (effects (font (size 1.27 1.27)))
+    )
+    (property "Value" "10K" (at 204.47 185.42 90)
+      (effects (font (size 1.27 1.27)))
+    )
+    (property "Footprint" "Resistor_SMD:R_0805_2012Metric" (at 204.47 187.96 0)
+      (effects (font (size 1.27 1.27)) hide)
+    )
+    (property "Datasheet" "~" (at 204.47 187.96 0)
+      (effects (font (size 1.27 1.27)) hide)
+    )
+    (pin "2")
+    (pin "1")
+    (instances
+      (project "GVH-POR-SpaceSuitScanner"
+        (path "/d220c84c-6011-402a-bba2-62b84e1ad1c6"
+          (reference "R5") (unit 1)
+        )
+      )
+    )
+  )
   (symbol (lib_id "power:GND") (at 121.92 177.8 0) (unit 1)
     (in_bom yes) (on_board yes) (dnp no) (fields_autoplaced)
@@
     )
   )
-  (symbol (lib_id "Device:R_Small") (at 161.29 195.58 270) (unit 1)
+  (symbol (lib_id "Device:R_Small") (at 161.29 198.12 270) (unit 1)
     (in_bom yes) (on_board yes) (dnp no)
-    (property "Reference" "R4" (at 161.29 190.5 90)
+    (property "Reference" "R4" (at 161.29 193.04 90)
       (effects (font (size 1.27 1.27)))
     )
-    (property "Value" "1K" (at 161.29 193.04 90)
+    (property "Value" "1K" (at 161.29 195.58 90)
       (effects (font (size 1.27 1.27)))
     )
-    (property "Footprint" "Resistor_SMD:R_0805_2012Metric" (at 161.29 195.58 0)
+    (property "Footprint" "Resistor_SMD:R_0805_2012Metric" (at 161.29 198.12 0)
       (effects (font (size 1.27 1.27)) hide)
     )
-    (property "Datasheet" "~" (at 161.29 195.58 0)
+    (property "Datasheet" "~" (at 161.29 198.12 0)
       (effects (font (size 1.27 1.27)) hide)
     )

Commit message: Added silkscreen graphics and signature. Ready for fab.
Other:
- title: Darlu Frill's Space Suit Hand Scan Activator -> Darlu's Spacesuit Activator
Changed lines of the file:
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@@
   (paper "USLedger")
   (title_block
-    (title "Darlu Frill's Space Suit Hand Scan Activator")
+    (title "Darlu's Spacesuit Activator")
     (date "2024-07-23")
     (rev "v0.1")

Commit message: Changed the library symbols to be project specific
Parts:
- C1, C2, C3, C4, R1, R2: Package (none) -> 0805; now not fitted; now left out of the parts list
- C5: Digikey P/N (none) -> 311-1138-1-ND; Digikey Page (none) -> https://www.digikey.com/en/products/detail/yageo/CC0805KRX7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; Package (none) -> 0805
- C6: Digikey P/N (none) -> 311-1140-1-ND; Digikey Page (none) -> https://www.digikey.com/en/products/detail/yageo/CC0805KRX7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; Package (none) -> 0805
- D1: value LED_Small -> Touch_Indicator; Digikey P/N (none) -> 160-1423-1-ND; Digikey Page (none) -> https://www.digikey.com/en/products/detail/liteon/LTST-C171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; Package (none) -> 0805
- D4: value LED_Small -> Rectangular_Green_LED; Digikey P/N (none) -> 754-WP113CGKDT-ND; Digikey Page (none) -> https://www.digikey.com/en/products/detail/kingbright/WP113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; Package (none) -> 5.00mm x 2.00mm Rectangular
- D5: value LED_Small -> Rectangular_Red_LED; Digikey P/N (none) -> 754-WP113SURDKT-ND; Digikey Page (none) -> https://www.digikey.com/en/products/detail/kingbright/WP113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; Package (none) -> 5.00mm x 2.00mm Rectangular
- J1, J11, J12, J13, J14, J15, J16, J17, J18, J2, J3, J4, J5, J6, J7, J8, J9: footprint my_footprints:PHOENIX_1725656-2POS -> 0_connector:PHOENIX_1725656-2POS; symbol my_library:Phoenix_2POS_725656 -> 0_connector:Phoenix_2POS_725656
- J10: footprint my_footprints:PHOENIX_1725685-5POS -> 0_connector:PHOENIX_1725685-5POS; symbol my_library:Phoenix_5POS_1725685 -> 0_connector:Phoenix_5POS_1725685
- J19: footprint my_footprints:PHOENIX_1725669-3POS -> 0_connector:PHOENIX_1725669-3POS; symbol my_library:Phoenix_3POS_1725669 -> 0_connector:Phoenix_3POS_1725669
- J29, J30: footprint my_footprints:MOLEX_MICROFIT-RA-4POS -> 0_connector:MOLEX_MICROFIT-RA-4POS; symbol my_library:Molex Micro-Fit 4pos -> 0_connector:Molex Micro-Fit 4pos
- J31: footprint my_footprints:MOLEX_MICROFIT-RA-2POS -> 0_connector:MOLEX_MICROFIT-RA-2POS; symbol my_library:Molex Micro-Fit 2pos -> 0_connector:Molex Micro-Fit 2pos
- JP1: value SolderJumper_2_Open -> R8_Bypass
- JP2: value SolderJumper_2_Open -> R9_Bypass
- R3, R5: Digikey P/N (none) -> 311-10.0KCRCT-ND; Digikey Page (none) -> https://www.digikey.com/en/products/detail/yageo/RC0805FR-0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; Package (none) -> 0805
- R4: Digikey P/N (none) -> 311-1.00KCRCT-ND; Digikey Page (none) -> https://www.digikey.com/en/products/detail/yageo/RC0805FR-0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; Package (none) -> 0805
- R8, R9: Digikey P/N (none) -> A129741CT-ND; Digikey Page (none) -> https://www.digikey.com/en/products/detail/te-connectivity-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; Package (none) -> 0805
- U1, U2: now not fitted; now left out of the parts list
- U3, U4: footprint my_footprints:Adafruit_AW9523_GPIO_Expander -> 0_breakout_board:Adafruit_AW9523_GPIO_Expander; symbol my_library:Adafruit_AW9523_GPIO_Expander -> 0_breakout_board:Adafruit_AW9523_GPIO_Expander
- U5: footprint my_footprints:SOT95P270X145-6N -> 0_sensor:AT42QT1010-TSGR_1; symbol my_library:AT42QT1010-TSHR_1 -> 0_sensor:AT42QT1010-TSHR_1
- U6: footprint my_footprints:Adafruit IS31FL3731 LED Driver -> 0_breakout_board:Adafruit IS31FL3731 LED Driver; symbol my_library:Adafruit_IS31FL3731_Matrix -> 0_breakout_board:Adafruit_IS31FL3731_Matrix
Other:
- note added: "THT Cap for adjusting sensitivity Not required"
- note removed: "THT Cap for adjusting sensitivity"
- moved on the sheet: D4, D5, R5
